Commit message: save: before adding 3rd leg

File: urdf/leg.xacro (robot description, xacro)
@@ -5,32 +5,13 @@
     <!-- xyz describes translation in meters -->
   <link name="${prefix}_leg">
-    <collision>
-      <origin xyz="0 0 ${-leg_height/2 - axel_offset}" rpy="0 0 0"/>
+    <visual>
+      <origin xyz="0 0 ${-leg_height/10 - axel_offset}" rpy="0 0 0"/>
       <geometry>
-	      <box size="${leg_width} ${leg_width} ${leg_height}"/>
-      </geometry>
-      <surface>
-        <friction>
-          <ode>
-            <mu>10000.0</mu>
-            <mu2>10000.0</mu2>
-          </ode>
-        </friction>
-        <contact>
-          <ode>
-            <min_depth>0.03</min_depth>
-          </ode>
-        </contact>
-      </surface>
-    </collision>
-    <visual>
-      <origin xyz="0 0 ${-leg_height/2 - axel_offset}" rpy="0 0 0"/>
-      <geometry>
-	      <box size="${leg_width} ${leg_width} ${leg_height}"/>
+	      <box size="${leg_width} ${leg_width} ${leg_height/5}"/>
       </geometry>
       <material name="orange"/>
     </visual>
     <inertial>
-      <origin xyz="0 0 ${-leg_height/2 - axel_offset}" rpy="0 0 0"/>
+      <origin xyz="0 0 ${-leg_height/10 - axel_offset}" rpy="0 0 0"/>
       <mass value="${mass/10}"/>
       <inertia ixx="0.06" ixy="0.0" ixz="0.0" iyy="0.06" iyz="0.0" izz="0.25"/>
@@ -40,5 +21,6 @@
     <parent link="base_link"/>
     <child link="${prefix}_leg"/>
-    <origin xyz="${position * robot_body_width} ${reflect * robot_body_width/2} ${start_height + robot_body_height/2 - axel_offset}" rpy="${1 * PI/3} 0 ${mirror * PI}"/>
+    <origin xyz="${position * robot_body_width} ${reflect * robot_body_width/2}
+    ${start_height + robot_body_height/2 - axel_offset}" rpy="${1 * PI/2} 0 ${mirror * PI}"/>
     <axis xyz="1 0 0"/>
     <limit effort="30" lower="${-PI/6}" upper="${PI/6}" velocity="1"/>
@@ -46,23 +28,4 @@
   <!-- leg_1_link_2 -->
   <link name="${prefix}_leg_link_2">
-    <collision>
-      <origin xyz="${leg_width/2} 0 ${-leg_height/2 + leg_width/2}" rpy="0 0 0"/>
-      <geometry>
-	      <box size="${leg_width} ${leg_width} ${leg_height}"/>
-      </geometry>
-      <surface>
-        <friction>
-          <ode>
-            <mu>10000.0</mu>
-            <mu2>10000.0</mu2>
-          </ode>
-        </friction>
-        <contact>
-          <ode>
-            <min_depth>0.03</min_depth>
-          </ode>
-        </contact>
-      </surface>
-    </collision>
     <visual>
       <origin xyz="${leg_width/2} 0 ${-leg_height/2 + leg_width/2}" rpy="0 0 0"/>
@@ -81,5 +44,6 @@
     <parent link="${prefix}_leg"/>
     <child link="${prefix}_leg_link_2"/>
-    <origin xyz="${leg_width/2} 0 ${-leg_height + leg_width/2}" rpy="${-PI/3} 0 0"/>
+    <origin xyz="${leg_width/2 - (mirror * leg_width)} 0 ${-leg_height/5 + leg_width/2 - axel_offset}" rpy="0 0 ${mirror * PI}"/>
+    <!-- <origin xyz="${leg_width/2} 0 ${-leg_height + leg_width/2}" rpy="3pi/2 0 0"/> -->
     <axis xyz="1 0 0"/>
     <limit effort="30" velocity="0.03"/>

File: urdf/main.xacro (robot description, xacro)
@@ -31,6 +31,10 @@
         </collision>
         <inertial>
+            <origin xyz="0 0 ${robot_body_height/2 + start_height}" rpy="0 0 0"/>
             <mass value="${mass}"/>
-            <inertia ixx="0.21" ixy="0" ixz="0" iyy="0.27" iyz="0" izz="0.10"/>
+                  <inertia
+	  ixx="${mass / 12.0 * (robot_body_height*robot_body_height + robot_body_width*robot_body_width)}" ixy="0.0" ixz="0.0"
+	  iyy="${mass / 12.0 * (robot_body_height*robot_body_height + (robot_body_width*3)*(3*robot_body_width))}" iyz="0.0"
+	  izz="${mass / 12.0 * (robot_body_width*robot_body_width + (robot_body_width*3)*(3*robot_body_width))}"/>
         </inertial>
     </link>
