Commit message: save: not fly away finally!

File: urdf/constants.xacro (robot description, xacro)
@@ -3,7 +3,7 @@
   <!-- Constants for robot dimensions -->
   <xacro:property name="PI" value="3.1415926535897931"/>
-  <xacro:property name="mass" value="10" /> <!-- arbitrary value for mass -->
+  <xacro:property name="mass" value="1" /> <!-- arbitrary value for mass -->
   <xacro:property name="robot_body_width" value="1" /> <!-- Square dimensions (widthxwidth) of beams -->
-  <xacro:property name="start_height" value="2" /> <!-- Square dimensions (widthxwidth) of beams -->
+  <xacro:property name="start_height" value="1.1" /> <!-- Square dimensions (widthxwidth) of beams -->
   <xacro:property name="leg_width" value="0.1" />
   <xacro:property name="robot_body_height" value="0.3" /> <!-- Link 1 -->

File: urdf/leg.xacro (robot description, xacro)
@@ -5,4 +5,10 @@
     <!-- xyz describes translation in meters -->
   <link name="${prefix}_leg">
+    <collision>
+      <origin xyz="0 0 ${-leg_height/10 - axel_offset}" rpy="0 0 0"/>
+      <geometry>
+	      <box size="${leg_width} ${leg_width} ${leg_height/5}"/>
+      </geometry>
+    </collision>
     <visual>
       <origin xyz="0 0 ${-leg_height/10 - axel_offset}" rpy="0 0 0"/>
@@ -14,6 +20,9 @@
     <inertial>
       <origin xyz="0 0 ${-leg_height/10 - axel_offset}" rpy="0 0 0"/>
-      <mass value="${mass/10}"/>
-      <inertia ixx="0.06" ixy="0.0" ixz="0.0" iyy="0.06" iyz="0.0" izz="0.25"/>
+      <mass value="${mass}"/>
+      <inertia
+	  ixx="1.0" ixy="0.0" ixz="0.0"
+	  iyy="1.0" iyz="0.0"
+	  izz="1.0"/>
     </inertial>
   </link>
@@ -24,8 +33,15 @@
     ${start_height + robot_body_height/2 - axel_offset}" rpy="${1 * PI/2} 0 ${mirror * PI}"/>
     <axis xyz="1 0 0"/>
-    <limit effort="30" lower="${-PI/6}" upper="${PI/6}" velocity="1"/>
+    <limit effort="30" velocity="0.1"/>
+    <dynamics damping="0.7" friction="0.1"/>
   </joint>
-  <!-- leg_1_link_2 -->
-  <link name="${prefix}_leg_link_2">
+  <!-- leg_1_link_1 -->
+  <link name="${prefix}_leg_link_1">
+    <collision>
+      <origin xyz="${leg_width/2} 0 ${-leg_height/2 + leg_width/2}" rpy="0 0 0"/>
+      <geometry>
+	      <box size="${leg_width} ${leg_width} ${leg_height}"/>
+      </geometry>
+    </collision>
     <visual>
       <origin xyz="${leg_width/2} 0 ${-leg_height/2 + leg_width/2}" rpy="0 0 0"/>
@@ -37,15 +53,52 @@
     <inertial>
       <origin xyz="${leg_width/2} 0 ${-leg_height/2 + leg_width/2}" rpy="0 0 0"/>
-      <mass value="${mass/10}"/>
-      <inertia ixx="0.06" ixy="0.0" ixz="0.0" iyy="0.06" iyz="0.0" izz="0.25"/>
+      <mass value="${mass}"/>
+      <inertia
+	  ixx="1.0" ixy="0.0" ixz="0.0"
+	  iyy="1.0" iyz="0.0"
+	  izz="1.0"/>
     </inertial>
   </link>
   <joint name="${prefix}_leg_joint_2" type="continuous">
     <parent link="${prefix}_leg"/>
-    <child link="${prefix}_leg_link_2"/>
+    <child link="${prefix}_leg_link_1"/>
     <origin xyz="${leg_width/2 - (mirror * leg_width)} 0 ${-leg_height/5 + leg_width/2 - axel_offset}" rpy="0 0 ${mirror * PI}"/>
     <!-- <origin xyz="${leg_width/2} 0 ${-leg_height + leg_width/2}" rpy="3pi/2 0 0"/> -->
     <axis xyz="1 0 0"/>
     <limit effort="30" velocity="0.03"/>
+    <dynamics damping="0.7" friction="0.1"/>
+  </joint>
+  <!-- leg_1_link_2 -->
+  <link name="${prefix}_leg_link_2">
+    <collision>
+      <origin xyz="${leg_width/2} 0 ${-leg_height/2 + leg_width/2}" rpy="0 0 0"/>
+      <geometry>
+	      <box size="${leg_width} ${leg_width} ${leg_height}"/>
+      </geometry>
+    </collision>
+    <visual>
+      <origin xyz="${leg_width/2} 0 ${-leg_height/2 + leg_width/2}" rpy="0 0 0"/>
+      <geometry>
+	      <box size="${leg_width} ${leg_width} ${leg_height}"/>
+      </geometry>
+      <material name="orange"/>
+    </visual>
+    <inertial>
+      <origin xyz="${leg_width/2} 0 ${-leg_height/2 + leg_width/2}" rpy="0 0 0"/>
+      <mass value="${mass}"/>
+      <inertia
+	  ixx="1.0" ixy="0.0" ixz="0.0"
+	  iyy="1.0" iyz="0.0"
+	  izz="1.0"/>
+    </inertial>
+  </link>
+  <joint name="${prefix}_leg_joint_3" type="continuous">
+    <parent link="${prefix}_leg_link_1"/>
+    <child link="${prefix}_leg_link_2"/>
+    <origin xyz="${-leg_width} 0 ${-leg_height + leg_width}" rpy="${-PI/2 + (mirror * PI)} 0 0"/>
+    <!-- <origin xyz="${leg_width/2} 0 ${-leg_height + leg_width/2}" rpy="3pi/2 0 0"/> -->
+    <axis xyz="1 0 0"/>
+    <limit effort="30" velocity="0.03"/>
+    <dynamics damping="0.7" friction="0.1"/>
   </joint>
     <transmission name="${prefix}_leg_transmission_1">
@@ -67,4 +120,37 @@
         </joint>
     </transmission>
+    <transmission name="${prefix}_leg_transmission_3">
+        <type>transmission_interface/SimpleTransmission</type>
+        <actuator name="$${prefix}_motor_3">
+            <mechanicalReduction>1</mechanicalReduction>
+        </actuator>
+        <joint name="${prefix}_leg_joint_3">
+            <hardwareInterface>hardware_interface/PositionJointInterface</hardwareInterface>
+        </joint>
+    </transmission>
+<gazebo reference="${prefix}_leg_joint_1">
+  <kp>1000000.0</kp>
+  <kd>1.0</kd>
+  <mu1>0.8</mu1>
+  <mu2>0.8</mu2>
+  <maxVel>0.0</maxVel>
+  <minDepth>0.001</minDepth>
+</gazebo>
+<gazebo reference="${prefix}_leg_joint_2">
+  <kp>1000000.0</kp>
+  <kd>1.0</kd>
+  <mu1>0.8</mu1>
+  <mu2>0.8</mu2>
+  <maxVel>0.0</maxVel>
+  <minDepth>0.001</minDepth>
+</gazebo>
+<gazebo reference="${prefix}_leg_joint_3">
+  <kp>1000000.0</kp>
+  <kd>1.0</kd>
+  <mu1>0.8</mu1>
+  <mu2>0.8</mu2>
+  <maxVel>0.0</maxVel>
+  <minDepth>0.001</minDepth>
+</gazebo>
 </xacro:macro>
 </robot>

Commit message: save: (kind of) able to walking now

File: urdf/constants.xacro (robot description, xacro)
@@ -3,8 +3,8 @@
   <!-- Constants for robot dimensions -->
   <xacro:property name="PI" value="3.1415926535897931"/>
-  <xacro:property name="mass" value="1" /> <!-- arbitrary value for mass -->
+  <xacro:property name="mass" value="0.1" /> <!-- arbitrary value for mass -->
   <xacro:property name="robot_body_width" value="1" /> <!-- Square dimensions (widthxwidth) of beams -->
   <xacro:property name="start_height" value="1.1" /> <!-- Square dimensions (widthxwidth) of beams -->
-  <xacro:property name="leg_width" value="0.1" />
+  <xacro:property name="leg_width" value="0.2" />
   <xacro:property name="robot_body_height" value="0.3" /> <!-- Link 1 -->
   <xacro:property name="leg_height" value="1" /> <!-- Link 2 -->

File: urdf/leg.xacro (robot description, xacro)
@@ -22,7 +22,73 @@
       <mass value="${mass}"/>
       <inertia
+	  ixx="${mass / 12.0 * (leg_width*leg_width + leg_height*leg_height/25)}" ixy="0.0" ixz="0.0"
+	  iyy="${mass / 12.0 * (leg_height*leg_height/25 + leg_width*leg_width)}" iyz="0.0"
+	  izz="${mass / 12.0 * (leg_width*leg_width + leg_width*leg_width)}"/>
+    <!--
+      <inertia
 	  ixx="1.0" ixy="0.0" ixz="0.0"
 	  iyy="1.0" iyz="0.0"
 	  izz="1.0"/>
+    -->
+      </inertial>
+  </link>
+  <!-- leg_1_link_1 -->
+  <link name="${prefix}_leg_link_1">
+    <collision>
+      <origin xyz="${leg_width/2 + axel_offset} 0 ${-leg_height/2 + leg_width/2}" rpy="0 0 0"/>
+      <geometry>
+	      <box size="${leg_width} ${leg_width} ${leg_height}"/>
+      </geometry>
+    </collision>
+    <visual>
+      <origin xyz="${leg_width/2 + axel_offset} 0 ${-leg_height/2 + leg_width/2}" rpy="0 0 0"/>
+      <geometry>
+	      <box size="${leg_width} ${leg_width} ${leg_height}"/>
+      </geometry>
+      <material name="orange"/>
+    </visual>
+    <inertial>
+      <origin xyz="${leg_width/2 + axel_offset} 0 ${-leg_height/2 + leg_width/2}" rpy="0 0 0"/>
+      <mass value="${mass}"/>
+      <inertia
+	  ixx="${mass / 12.0 * (leg_width*leg_width + leg_height*leg_height)}" ixy="0.0" ixz="0.0"
+	  iyy="${mass / 12.0 * (leg_height*leg_height + leg_width*leg_width)}" iyz="0.0"
+	  izz="${mass / 12.0 * (leg_width*leg_width + leg_width*leg_width)}"/>
+    <!--
+      <inertia
+	  ixx="1.0" ixy="0.0" ixz="0.0"
+	  iyy="1.0" iyz="0.0"
+	  izz="1.0"/>
+    -->
+    </inertial>
+  </link>
+  <!-- leg_1_link_2 -->
+  <link name="${prefix}_leg_link_2">
+    <collision>
+      <origin xyz="${leg_width/2 + axel_offset} 0 ${-leg_height/2 + leg_width/2}" rpy="0 0 0"/>
+      <geometry>
+	      <box size="${leg_width} ${leg_width} ${leg_height}"/>
+      </geometry>
+    </collision>
+    <visual>
+      <origin xyz="${leg_width/2 + axel_offset} 0 ${-leg_height/2 + leg_width/2}" rpy="0 0 0"/>
+      <geometry>
+	      <box size="${leg_width} ${leg_width} ${leg_height}"/>
+      </geometry>
+      <material name="orange"/>
+    </visual>
+    <inertial>
+      <origin xyz="${leg_width/2 + axel_offset} 0 ${-leg_height/2 + leg_width/2}" rpy="0 0 0"/>
+      <mass value="${mass}"/>
+      <inertia
+	  ixx="${mass / 12.0 * (leg_width*leg_width + leg_height*leg_height)}" ixy="0.0" ixz="0.0"
+	  iyy="${mass / 12.0 * (leg_height*leg_height + leg_width*leg_width)}" iyz="0.0"
+	  izz="${mass / 12.0 * (leg_width*leg_width + leg_width*leg_width)}"/>
+    <!--
+      <inertia
+	  ixx="1.0" ixy="0.0" ixz="0.0"
+	  iyy="1.0" iyz="0.0"
+	  izz="1.0"/>
+    -->
     </inertial>
   </link>
@@ -32,32 +98,7 @@
     <origin xyz="${position * robot_body_width} ${reflect * robot_body_width/2}
     ${start_height + robot_body_height/2 - axel_offset}" rpy="${1 * PI/2} 0 ${mirror * PI}"/>
-    <axis xyz="1 0 0"/>
-    <limit effort="30" velocity="0.1"/>
-    <dynamics damping="0.7" friction="0.1"/>
+    <axis xyz="0 1 0"/>
+    <limit effort="1000" velocity="0.5"/>
   </joint>
-  <!-- leg_1_link_1 -->
-  <link name="${prefix}_leg_link_1">
-    <collision>
-      <origin xyz="${leg_width/2} 0 ${-leg_height/2 + leg_width/2}" rpy="0 0 0"/>
-      <geometry>
-	      <box size="${leg_width} ${leg_width} ${leg_height}"/>
-      </geometry>
-    </collision>
-    <visual>
-      <origin xyz="${leg_width/2} 0 ${-leg_height/2 + leg_width/2}" rpy="0 0 0"/>
-      <geometry>
-	      <box size="${leg_width} ${leg_width} ${leg_height}"/>
-      </geometry>
-      <material name="orange"/>
-    </visual>
-    <inertial>
-      <origin xyz="${leg_width/2} 0 ${-leg_height/2 + leg_width/2}" rpy="0 0 0"/>
-      <mass value="${mass}"/>
-      <inertia
-	  ixx="1.0" ixy="0.0" ixz="0.0"
-	  iyy="1.0" iyz="0.0"
-	  izz="1.0"/>
-    </inertial>
-  </link>
   <joint name="${prefix}_leg_joint_2" type="continuous">
     <parent link="${prefix}_leg"/>
@@ -66,39 +107,13 @@
     <!-- <origin xyz="${leg_width/2} 0 ${-leg_height + leg_width/2}" rpy="3pi/2 0 0"/> -->
     <axis xyz="1 0 0"/>
-    <limit effort="30" velocity="0.03"/>
-    <dynamics damping="0.7" friction="0.1"/>
+    <limit effort="1000" velocity="0.5"/>
   </joint>
-  <!-- leg_1_link_2 -->
-  <link name="${prefix}_leg_link_2">
-    <collision>
-      <origin xyz="${leg_width/2} 0 ${-leg_height/2 + leg_width/2}" rpy="0 0 0"/>
-      <geometry>
-	      <box size="${leg_width} ${leg_width} ${leg_height}"/>
-      </geometry>
-    </collision>
-    <visual>
-      <origin xyz="${leg_width/2} 0 ${-leg_height/2 + leg_width/2}" rpy="0 0 0"/>
-      <geometry>
-	      <box size="${leg_width} ${leg_width} ${leg_height}"/>
-      </geometry>
-      <material name="orange"/>
-    </visual>
-    <inertial>
-      <origin xyz="${leg_width/2} 0 ${-leg_height/2 + leg_width/2}" rpy="0 0 0"/>
-      <mass value="${mass}"/>
-      <inertia
-	  ixx="1.0" ixy="0.0" ixz="0.0"
-	  iyy="1.0" iyz="0.0"
-	  izz="1.0"/>
-    </inertial>
-  </link>
   <joint name="${prefix}_leg_joint_3" type="continuous">
     <parent link="${prefix}_leg_link_1"/>
     <child link="${prefix}_leg_link_2"/>
-    <origin xyz="${-leg_width} 0 ${-leg_height + leg_width}" rpy="${-PI/2 + (mirror * PI)} 0 0"/>
+    <origin xyz="${axel_offset} 0 ${-leg_height + leg_width}" rpy="${-PI/2 + (mirror * PI)} ${PI} 0"/>
     <!-- <origin xyz="${leg_width/2} 0 ${-leg_height + leg_width/2}" rpy="3pi/2 0 0"/> -->
     <axis xyz="1 0 0"/>
-    <limit effort="30" velocity="0.03"/>
-    <dynamics damping="0.7" friction="0.1"/>
+    <limit effort="1000" velocity="0.5"/>
   </joint>
     <transmission name="${prefix}_leg_transmission_1">
@@ -129,5 +144,5 @@
         </joint>
     </transmission>
-<gazebo reference="${prefix}_leg_joint_1">
+<gazebo reference="${prefix}_leg">
   <kp>1000000.0</kp>
   <kd>1.0</kd>
@@ -137,5 +152,5 @@
   <minDepth>0.001</minDepth>
 </gazebo>
-<gazebo reference="${prefix}_leg_joint_2">
+<gazebo reference="${prefix}_leg_link_1">
   <kp>1000000.0</kp>
   <kd>1.0</kd>
@@ -145,5 +160,5 @@
   <minDepth>0.001</minDepth>
 </gazebo>
-<gazebo reference="${prefix}_leg_joint_3">
+<gazebo reference="${prefix}_leg_link_2">
   <kp>1000000.0</kp>
   <kd>1.0</kd>

File: urdf/main.xacro (robot description, xacro)
@@ -39,4 +39,12 @@
         </inertial>
     </link>
+<gazebo reference="base_link">
+  <kp>1000000.0</kp>
+  <kd>1.0</kd>
+  <mu1>0.8</mu1>
+  <mu2>0.8</mu2>
+  <maxVel>0.0</maxVel>
+  <minDepth>0.001</minDepth>
+</gazebo>
     <xacro:leg prefix="left_back" position="-1" reflect="1" mirror="0" />
     <xacro:leg prefix="left_mid" position="0" reflect="1" mirror="0" />

Commit message: save: upgraded but still lackluster moving

File: urdf/constants.xacro (robot description, xacro)
@@ -3,7 +3,7 @@
   <!-- Constants for robot dimensions -->
   <xacro:property name="PI" value="3.1415926535897931"/>
-  <xacro:property name="mass" value="0.1" /> <!-- arbitrary value for mass -->
+  <xacro:property name="mass" value="0.01" /> <!-- arbitrary value for mass -->
   <xacro:property name="robot_body_width" value="1" /> <!-- Square dimensions (widthxwidth) of beams -->
-  <xacro:property name="start_height" value="1.1" /> <!-- Square dimensions (widthxwidth) of beams -->
+  <xacro:property name="start_height" value="0.7" /> <!-- Square dimensions (widthxwidth) of beams -->
   <xacro:property name="leg_width" value="0.2" />
   <xacro:property name="robot_body_height" value="0.3" /> <!-- Link 1 -->

File: urdf/leg.xacro (robot description, xacro)
@@ -33,6 +33,35 @@
       </inertial>
   </link>
-  <!-- leg_1_link_1 -->
   <link name="${prefix}_leg_link_1">
+    <collision>
+      <origin xyz="0 0 ${-leg_height/10 - axel_offset}" rpy="0 0 0"/>
+      <geometry>
+	      <box size="${leg_width} ${leg_width} ${leg_height/5}"/>
+      </geometry>
+    </collision>
+    <visual>
+      <origin xyz="0 0 ${-leg_height/10 - axel_offset}" rpy="0 0 0"/>
+      <geometry>
+	      <box size="${leg_width} ${leg_width} ${leg_height/5}"/>
+      </geometry>
+      <material name="orange"/>
+    </visual>
+    <inertial>
+      <origin xyz="0 0 ${-leg_height/10 - axel_offset}" rpy="0 0 0"/>
+      <mass value="${mass}"/>
+      <inertia
+	  ixx="${mass / 12.0 * (leg_width*leg_width + leg_height*leg_height/25)}" ixy="0.0" ixz="0.0"
+	  iyy="${mass / 12.0 * (leg_height*leg_height/25 + leg_width*leg_width)}" iyz="0.0"
+	  izz="${mass / 12.0 * (leg_width*leg_width + leg_width*leg_width)}"/>
+    <!--
+      <inertia
+	  ixx="1.0" ixy="0.0" ixz="0.0"
+	  iyy="1.0" iyz="0.0"
+	  izz="1.0"/>
+    -->
+      </inertial>
+  </link>
+  <!-- leg_1_link_2 -->
+  <link name="${prefix}_leg_link_2">
     <collision>
       <origin xyz="${leg_width/2 + axel_offset} 0 ${-leg_height/2 + leg_width/2}" rpy="0 0 0"/>
@@ -63,6 +92,6 @@
     </inertial>
   </link>
-  <!-- leg_1_link_2 -->
-  <link name="${prefix}_leg_link_2">
+  <!-- leg_1_link_3 -->
+  <link name="${prefix}_leg_link_3">
     <collision>
       <origin xyz="${leg_width/2 + axel_offset} 0 ${-leg_height/2 + leg_width/2}" rpy="0 0 0"/>
@@ -104,7 +133,7 @@
     <parent link="${prefix}_leg"/>
     <child link="${prefix}_leg_link_1"/>
-    <origin xyz="${leg_width/2 - (mirror * leg_width)} 0 ${-leg_height/5 + leg_width/2 - axel_offset}" rpy="0 0 ${mirror * PI}"/>
+    <origin xyz="0 0 ${-leg_height/5 - axel_offset}" rpy="0 0 0"/>
     <!-- <origin xyz="${leg_width/2} 0 ${-leg_height + leg_width/2}" rpy="3pi/2 0 0"/> -->
-    <axis xyz="1 0 0"/>
+    <axis xyz="0 0 1"/>
     <limit effort="1000" velocity="0.5"/>
   </joint>
@@ -112,4 +141,12 @@
     <parent link="${prefix}_leg_link_1"/>
     <child link="${prefix}_leg_link_2"/>
+    <origin xyz="${leg_width/2 - (mirror * leg_width)} 0 ${-leg_height/5 + leg_width/2 - axel_offset}" rpy="${PI/8 - (mirror * PI/4)} 0 ${mirror * PI}"/>
+    <!-- <origin xyz="${leg_width/2} 0 ${-leg_height + leg_width/2}" rpy="3pi/2 0 0"/> -->
+    <axis xyz="1 0 0"/>
+    <limit effort="1000" velocity="0.5"/>
+  </joint>
+  <joint name="${prefix}_leg_joint_4" type="continuous">
+    <parent link="${prefix}_leg_link_2"/>
+    <child link="${prefix}_leg_link_3"/>
     <origin xyz="${axel_offset} 0 ${-leg_height + leg_width}" rpy="${-PI/2 + (mirror * PI)} ${PI} 0"/>
     <!-- <origin xyz="${leg_width/2} 0 ${-leg_height + leg_width/2}" rpy="3pi/2 0 0"/> -->
@@ -144,27 +181,53 @@
         </joint>
     </transmission>
+    <transmission name="${prefix}_leg_transmission_4">
+        <type>transmission_interface/SimpleTransmission</type>
+        <actuator name="$${prefix}_motor_4">
+            <mechanicalReduction>1</mechanicalReduction>
+        </actuator>
+        <joint name="${prefix}_leg_joint_4">
+            <hardwareInterface>hardware_interface/PositionJointInterface</hardwareInterface>
+        </joint>
+    </transmission>
 <gazebo reference="${prefix}_leg">
   <kp>1000000.0</kp>
   <kd>1.0</kd>
-  <mu1>0.8</mu1>
-  <mu2>0.8</mu2>
+  <mu1>1000</mu1>
+  <mu2>1000</mu2>
   <maxVel>0.0</maxVel>
   <minDepth>0.001</minDepth>
+  <fdir1>1 0 0</fdir1>
+  <material>Gazebo/Black</material>
 </gazebo>
 <gazebo reference="${prefix}_leg_link_1">
   <kp>1000000.0</kp>
   <kd>1.0</kd>
-  <mu1>0.8</mu1>
-  <mu2>0.8</mu2>
+  <mu1>1000</mu1>
+  <mu2>1000</mu2>
   <maxVel>0.0</maxVel>
   <minDepth>0.001</minDepth>
+  <fdir1>1 0 0</fdir1>
+  <material>Gazebo/Orange</material>
 </gazebo>
 <gazebo reference="${prefix}_leg_link_2">
   <kp>1000000.0</kp>
   <kd>1.0</kd>
-  <mu1>0.8</mu1>
-  <mu2>0.8</mu2>
+  <mu1>1000</mu1>
+  <mu2>1000</mu2>
   <maxVel>0.0</maxVel>
   <minDepth>0.001</minDepth>
+  <fdir1>1 0 0</fdir1>
+  <material>Gazebo/Black</material>
+</gazebo>
+<gazebo reference="${prefix}_leg_link_3">
+  <kp>1000000.0</kp>
+  <kd>100.0</kd>
+  <mu1>1.0</mu1>
+  <mu2>1.0</mu2>
+  <maxVel>1.0</maxVel>
+  <maxContacts>1</maxContacts>
+  <minDepth>0.001</minDepth>
+  <fdir1>1 0 0</fdir1>
+  <material>Gazebo/Orange</material>
 </gazebo>
 </xacro:macro>

File: urdf/main.xacro (robot description, xacro)
@@ -6,5 +6,5 @@
     <link name="base_link">
         <visual>
-            <origin xyz="0 0 ${robot_body_height/2 + start_height}" rpy="0 0 0"/>
+            <origin xyz="0 0 ${start_height}" rpy="0 0 0"/>
             <geometry>
                 <box size="${robot_body_width*3} ${robot_body_width} ${robot_body_height}"/>
@@ -12,5 +12,5 @@
         </visual>
         <collision>
-            <origin xyz="0 0 ${robot_body_height/2 + start_height}" rpy="0 0 0"/>
+            <origin xyz="0 0 ${start_height}" rpy="0 0 0"/>
             <geometry>
                 <box size="${robot_body_width*3} ${robot_body_width} ${robot_body_height}"/>
@@ -31,10 +31,10 @@
         </collision>
         <inertial>
-            <origin xyz="0 0 ${robot_body_height/2 + start_height}" rpy="0 0 0"/>
-            <mass value="${mass}"/>
+            <origin xyz="0 0 ${start_height}" rpy="0 0 0"/>
+            <mass value="${mass*10}"/>
                   <inertia
-	  ixx="${mass / 12.0 * (robot_body_height*robot_body_height + robot_body_width*robot_body_width)}" ixy="0.0" ixz="0.0"
-	  iyy="${mass / 12.0 * (robot_body_height*robot_body_height + (robot_body_width*3)*(3*robot_body_width))}" iyz="0.0"
-	  izz="${mass / 12.0 * (robot_body_width*robot_body_width + (robot_body_width*3)*(3*robot_body_width))}"/>
+	  ixx="${mass*10 / 12.0 * (robot_body_height*robot_body_height + robot_body_width*robot_body_width)}" ixy="0.0" ixz="0.0"
+	  iyy="${mass*10 / 12.0 * (robot_body_height*robot_body_height + (robot_body_width*3)*(3*robot_body_width))}" iyz="0.0"
+	  izz="${mass*10 / 12.0 * (robot_body_width*robot_body_width + (robot_body_width*3)*(3*robot_body_width))}"/>
         </inertial>
     </link>
@@ -46,4 +46,5 @@
   <maxVel>0.0</maxVel>
   <minDepth>0.001</minDepth>
+  <material>Gazebo/Orange</material>
 </gazebo>
     <xacro:leg prefix="left_back" position="-1" reflect="1" mirror="0" />
