Commit message: save: some minor changes (i guess)

File: urdf/constants.xacro (robot description, xacro)
@@ -5,5 +5,5 @@
   <xacro:property name="mass" value="0.01" /> <!-- arbitrary value for mass -->
   <xacro:property name="robot_body_width" value="1" /> <!-- Square dimensions (widthxwidth) of beams -->
-  <xacro:property name="start_height" value="0.7" /> <!-- Square dimensions (widthxwidth) of beams -->
+  <xacro:property name="start_height" value="0.0" /> <!-- Square dimensions (widthxwidth) of beams -->
   <xacro:property name="leg_width" value="0.2" />
   <xacro:property name="robot_body_height" value="0.3" /> <!-- Link 1 -->

File: urdf/leg.xacro (robot description, xacro)
@@ -99,4 +99,12 @@
 	      <box size="${leg_width} ${leg_width} ${leg_height}"/>
       </geometry>
+      <surface>
+        <friction>
+          <ode><mu>100000.0</mu><mu2>100000.0</mu2></ode>
+        </friction>
+                <contact>
+                  <ode><min_depth>0.003</min_depth></ode>
+                </contact>
+      </surface>
     </collision>
     <visual>
@@ -128,5 +136,5 @@
     ${start_height + robot_body_height/2 - axel_offset}" rpy="${1 * PI/2} 0 ${mirror * PI}"/>
     <axis xyz="0 1 0"/>
-    <limit effort="1000" velocity="0.5"/>
+    <limit effort="1000000" velocity="1"/>
   </joint>
   <joint name="${prefix}_leg_joint_2" type="continuous">
@@ -136,5 +144,5 @@
     <!-- <origin xyz="${leg_width/2} 0 ${-leg_height + leg_width/2}" rpy="3pi/2 0 0"/> -->
     <axis xyz="0 0 1"/>
-    <limit effort="1000" velocity="0.5"/>
+    <limit effort="1000000" velocity="1"/>
   </joint>
   <joint name="${prefix}_leg_joint_3" type="continuous">
@@ -144,13 +152,13 @@
     <!-- <origin xyz="${leg_width/2} 0 ${-leg_height + leg_width/2}" rpy="3pi/2 0 0"/> -->
     <axis xyz="1 0 0"/>
-    <limit effort="1000" velocity="0.5"/>
+    <limit effort="1000000" velocity="1"/>
   </joint>
   <joint name="${prefix}_leg_joint_4" type="continuous">
     <parent link="${prefix}_leg_link_2"/>
     <child link="${prefix}_leg_link_3"/>
-    <origin xyz="${axel_offset} 0 ${-leg_height + leg_width}" rpy="${-PI/2 + (mirror * PI)} ${PI} 0"/>
+    <origin xyz="${axel_offset} 0 ${-leg_height + leg_width}" rpy="${-3*PI/8 + (mirror * 6*PI/8)} ${PI} 0"/>
     <!-- <origin xyz="${leg_width/2} 0 ${-leg_height + leg_width/2}" rpy="3pi/2 0 0"/> -->
     <axis xyz="1 0 0"/>
-    <limit effort="1000" velocity="0.5"/>
+    <limit effort="1000000" velocity="1"/>
   </joint>
     <transmission name="${prefix}_leg_transmission_1">
@@ -221,12 +229,11 @@
 </gazebo>
 <gazebo reference="${prefix}_leg_link_3">
-  <kp>1000000.0</kp>
-  <kd>100.0</kd>
-  <mu1>1.0</mu1>
-  <mu2>1.0</mu2>
-  <maxVel>1.0</maxVel>
-  <maxContacts>1</maxContacts>
-  <minDepth>0.001</minDepth>
-  <fdir1>1 0 0</fdir1>
+    <kp>1000000.0</kp>
+    <kd>100.0</kd>
+    <mu1>10000.0</mu1>
+    <mu2>10000.0</mu2>
+    <fdir1>1 0 0</fdir1>
+    <maxVel>1.0</maxVel>
+    <minDepth>0.0001</minDepth>
   <material>Gazebo/Orange</material>
 </gazebo>

File: urdf/main.xacro (robot description, xacro)
@@ -25,5 +25,5 @@
               <contact>
                 <ode>
-                  <min_depth>0.03</min_depth>
+                  <min_depth>0.003</min_depth>
                 </ode>
               </contact>
